Commit message: postition and flange

File: man_gazebo/urdf/6dof/manipulator.urdf.xacro (robot description, xacro)
@@ -9,5 +9,5 @@
     <parent link="world" />
     <child link = "base_link" />
-    <origin xyz="0 -1 0" rpy="0.0 0.0 0.0" />
+    <origin xyz="0 0 0" rpy="0.0 0.0 0.0" />
   </joint>
   <xacro:macro name="cylinder_inertial" params="radius length mass *origin">
@@ -26,6 +26,6 @@
 	</xacro:if>
 	<xacro:unless value="${joint_type == 'revolute'}"  >
-		<xacro:property name="joint_upper_limit" value="${2*link_length}" />
-		<xacro:property name="joint_lower_limit" value="${0}" />
+		<xacro:property name="joint_upper_limit" value="${link_length}" />
+		<xacro:property name="joint_lower_limit" value="${-link_length}" />
 	</xacro:unless>
 	<limit lower="${joint_lower_limit}" upper="${joint_upper_limit}" effort="150.0" velocity="3.15"/>
@@ -39,5 +39,5 @@
 	<xacro:property name="joint5_type" value="revolute" />
 	<xacro:property name="joint6_type" value="revolute" />
-	<xacro:property name="joint0_axe" value="0 0 1" />
+	<xacro:property name="joint0_axe" value="0 1 0" />
 	<xacro:property name="joint1_axe" value="0 0 1" />
 	<xacro:property name="joint2_axe" value="0 1 0" />
@@ -56,6 +56,7 @@
 	<xacro:property name="link6_length" value="0.02" />
     <!-- Inertia parameters -->
-	<xacro:property name="link0_mass" value="40.7" />
-    <xacro:property name="base_mass" value="1.0" />
+    <xacro:property name="base_mass" value="44" />
+    <xacro:property name="ee_mass" value="2.5" />
+    <xacro:property name="link0_mass" value="7" />
     <xacro:property name="link1_mass" value="3.7" />
     <xacro:property name="link2_mass" value="8.393" />
@@ -86,7 +87,11 @@
         </geometry>
       </collision>
-      <xacro:cylinder_inertial radius="${base_radius}" length="${base_length}" mass="${base_mass}">
-        <origin xyz="0.0 0.0 ${base_length/2}" rpy="0 0 0" />
-      </xacro:cylinder_inertial>
+      <inertial>
+        <mass value="${base_mass}" />
+        <origin xyz="0.0 0.0 ${base_height/2}" />
+        <inertia ixx="436.5" ixy="0"  ixz="0"
+                          iyy="1.8" iyz="0"
+                                  izz="436.5"/>
+      </inertial>
     </link>
 <!--  joint 0	-->
@@ -96,5 +101,5 @@
       <origin xyz="0.0 0 ${base_height + link0_radius+0.01}" rpy="0 0.0 0" />
       <axis xyz="${joint0_axe}" />
-	  <xacro:joint_limit joint_type="${joint0_type}" link_length="${link0_length*6}"/>
+	  <xacro:joint_limit joint_type="${joint0_type}" link_length="${base_length/2}"/>
       <dynamics damping="0.0" friction="0.0"/>
     </joint>
@@ -280,5 +285,5 @@
     </link>
          <!-- fake joint - the rotation about z axe of the camera is not important -->
-        <joint name="fake_joint" type="revolute">
+   <!--  <joint name="fake_joint" type="revolute">
       <parent link="${prefix}link6" />
       <child link = "camera_link" />
@@ -287,7 +292,7 @@
       <xacro:joint_limit joint_type="revolute" link_length="0.1"/>
       <dynamics damping="0.0" friction="0.0"/>
-        </joint>
+    </joint> -->
     <!-- camera link -->
-        <link name="camera_link">
+    <!--     <link name="camera_link">
           <collision>
             <geometry>
@@ -300,6 +305,7 @@
           </xacro:cylinder_inertial>
         </link>
+ -->
     <joint name="${prefix}ee_fixed_joint" type="fixed">
-      <parent link="${prefix}camera_link" />
+      <parent link="${prefix}link6" />
       <child link = "${prefix}ee_link" />
       <origin xyz="0.0  0.0 0.01" rpy="0.0 0.0 0" />
@@ -307,4 +313,22 @@
 <!-- ee link -->
     <link name="${prefix}ee_link">
+      <visual>
+        <geometry>
+          <mesh filename="/home/student/catkin_ws/src/sock-puppet/man_gazebo/urdf/meshes/ee.dae" scale="0.0005 0.0005 0.0005" />
+        </geometry>
+      </visual>
+      <collision>
+        <geometry>
+          <mesh filename="/home/student/catkin_ws/src/sock-puppet/man_gazebo/urdf/meshes/ee.dae" scale="0.0005 0.0005 0.0005"/>
+        </geometry>
+      </collision>
+      <inertial>
+        <mass value="${ee_mass}" />
+        <origin xyz="0.0 0.0 ${base_height/2}" />
+        <inertia ixx="24.5" ixy="0"  ixz="0"
+                          iyy="0.1" iyz="0"
+                                  izz="24.5"/>
+      </inertial>
+<!--
       <collision>
         <geometry>
@@ -312,5 +336,5 @@
         </geometry>
         <origin rpy="0 0 0" xyz="0 0 0.005"/>
-      </collision>
+      </collision> -->
 	</link>
     <xacro:arm_transmission prefix="${prefix}" />
