Commit message: working simulation

File: man_code/scripts/roll_z_0_1pitch_z_0_7pitch_y_0_4pitch_x_0_7roll_z_0_1pitch_y_0_11.urdf.xacro (robot description, xacro)
@@ -39,9 +39,9 @@
         <xacro:property name="link0_mass" value="40.7" />
         <xacro:property name="link1_mass" value="3.7" />
-        <xacro:property name="link2_mass" value="10.89" />
-        <xacro:property name="link3_mass" value="2.63" />
-        <xacro:property name="link4_mass" value="7.04" />
+        <xacro:property name="link2_mass" value="10.45" />
+        <xacro:property name="link3_mass" value="3.51" />
+        <xacro:property name="link4_mass" value="6.16" />
         <xacro:property name="link5_mass" value="0.87" />
-        <xacro:property name="link6_mass" value="0.44" />
+        <xacro:property name="link6_mass" value="0.97" />
         <xacro:property name="link1_radius" value="0.049" />
         <xacro:property name="link2_radius" value="0.045" />
@@ -104,5 +104,5 @@
 <xacro:property name="joint1_type" value="revolute"/>
 <xacro:property name="joint1_axe" value="0 0 1"/>
-<xacro:property name="link1_length" value="0.44"/>
+<xacro:property name="link1_length" value="0.1"/>
 <!--  joint 1    -->
         <joint name="${prefix}joint1" type="${joint1_type}">
@@ -134,10 +134,10 @@
 <xacro:property name="joint2_type" value="revolute"/>
 <xacro:property name="joint2_axe" value="0 1 0"/>
-<xacro:property name="link2_length" value="0.75"/>
+<xacro:property name="link2_length" value="0.7"/>
 <!--  joint 2   -->
         <joint name="${prefix}joint2" type="${joint2_type}">
           <parent link="${prefix}link1"/>
           <child link="${prefix}link2" />
-          <origin xyz="0 ${link1_radius+link2_radius} ${link1_length}" rpy="0 0 0 "/>
+          <origin xyz="0 0 ${link1_length + link2_radius}" rpy="${1/2*pi} 0 0 "/>
           <axis xyz="${joint2_axe}"/>
           <xacro:joint_limit joint_type="${joint2_type}" link_length="${link2_length}"/>
@@ -164,5 +164,5 @@
 <xacro:property name="joint3_type" value="revolute"/>
 <xacro:property name="joint3_axe" value="0 1 0"/>
-<xacro:property name="link3_length" value="0.3"/>
+<xacro:property name="link3_length" value="0.4"/>
 <!--  joint 3   -->
         <joint name="${prefix}joint3" type="${joint3_type}">
@@ -194,10 +194,10 @@
 <xacro:property name="joint4_type" value="revolute"/>
 <xacro:property name="joint4_axe" value="0 1 0"/>
-<xacro:property name="link4_length" value="0.8"/>
+<xacro:property name="link4_length" value="0.7"/>
 <!--  joint 4   -->
         <joint name="${prefix}joint4" type="${joint4_type}">
           <parent link="${prefix}link3"/>
           <child link="${prefix}link4" />
-          <origin xyz="0 ${link3_radius+link4_radius} ${link3_length}" rpy="0 0 0 "/>
+          <origin xyz=" ${link3_radius+link4_radius} 0 ${link3_length}" rpy="0 0 ${-pi/2} "/>
           <axis xyz="${joint4_axe}"/>
           <xacro:joint_limit joint_type="${joint4_type}" link_length="${link4_length}"/>
@@ -254,5 +254,5 @@
 <xacro:property name="joint6_type" value="revolute"/>
 <xacro:property name="joint6_axe" value="0 1 0"/>
-<xacro:property name="link6_length" value="0.05"/>
+<xacro:property name="link6_length" value="0.11"/>
 <!--  joint 6   -->
         <joint name="${prefix}joint6" type="${joint6_type}">

File: man_gazebo/urdf/6dof/combined/pitch_x_0_1roll_z_0_7pitch_y_0_1pitch_x_0_4roll_z_0_1pitch_y_0_1.urdf.xacro (robot description, xacro)
@@ -36,12 +36,12 @@
         <xacro:property name="base_height"  value="0.5" />
             <!-- Inertia parameters -->
-        <xacro:property name="base_mass" value="1.0" />
-        <xacro:property name="link0_mass" value="40.7" />
+        <xacro:property name="base_mass" value="44" />
+        <xacro:property name="link0_mass" value="7" />
         <xacro:property name="link1_mass" value="3.7" />
-        <xacro:property name="link2_mass" value="10.89" />
-        <xacro:property name="link3_mass" value="2.63" />
-        <xacro:property name="link4_mass" value="7.04" />
-        <xacro:property name="link5_mass" value="0.87" />
-        <xacro:property name="link6_mass" value="0.62" />
+        <xacro:property name="link2_mass" value="10.45" />
+        <xacro:property name="link3_mass" value="0.88" />
+        <xacro:property name="link4_mass" value="3.51" />
+        <xacro:property name="link5_mass" value="0.88" />
+        <xacro:property name="link6_mass" value="0.88" />
         <xacro:property name="link1_radius" value="0.049" />
         <xacro:property name="link2_radius" value="0.045" />
@@ -104,5 +104,5 @@
 <xacro:property name="joint1_type" value="revolute"/>
 <xacro:property name="joint1_axe" value="0 1 0"/>
-<xacro:property name="link1_length" value="0.44"/>
+<xacro:property name="link1_length" value="0.1"/>
 <!--  joint 1    -->
         <joint name="${prefix}joint1" type="${joint1_type}">
@@ -133,11 +133,11 @@
         </link>
 <xacro:property name="joint2_type" value="revolute"/>
-<xacro:property name="joint2_axe" value="0 1 0"/>
-<xacro:property name="link2_length" value="0.75"/>
+<xacro:property name="joint2_axe" value="0 0 1"/>
+<xacro:property name="link2_length" value="0.7"/>
 <!--  joint 2   -->
         <joint name="${prefix}joint2" type="${joint2_type}">
           <parent link="${prefix}link1"/>
           <child link="${prefix}link2" />
-          <origin xyz="0 0 ${link1_length + link2_radius}" rpy="${-1/2*pi} 0 0 "/>
+          <origin xyz="0 0 ${link1_length}" rpy="0 0 0 "/>
           <axis xyz="${joint2_axe}"/>
           <xacro:joint_limit joint_type="${joint2_type}" link_length="${link2_length}"/>
@@ -164,5 +164,5 @@
 <xacro:property name="joint3_type" value="revolute"/>
 <xacro:property name="joint3_axe" value="0 1 0"/>
-<xacro:property name="link3_length" value="0.3"/>
+<xacro:property name="link3_length" value="0.1"/>
 <!--  joint 3   -->
         <joint name="${prefix}joint3" type="${joint3_type}">
@@ -194,5 +194,5 @@
 <xacro:property name="joint4_type" value="revolute"/>
 <xacro:property name="joint4_axe" value="0 1 0"/>
-<xacro:property name="link4_length" value="0.8"/>
+<xacro:property name="link4_length" value="0.4"/>
 <!--  joint 4   -->
         <joint name="${prefix}joint4" type="${joint4_type}">
@@ -254,5 +254,5 @@
 <xacro:property name="joint6_type" value="revolute"/>
 <xacro:property name="joint6_axe" value="0 1 0"/>
-<xacro:property name="link6_length" value="0.07"/>
+<xacro:property name="link6_length" value="0.1"/>
 <!--  joint 6   -->
         <joint name="${prefix}joint6" type="${joint6_type}">

File: man_gazebo/urdf/6dof/combined/pitch_z_0_1pitch_z_0_7pitch_y_0_4pitch_x_0_7roll_z_0_1pitch_y_0_1.urdf.xacro (robot description, xacro)
@@ -36,12 +36,12 @@
         <xacro:property name="base_height"  value="0.5" />
             <!-- Inertia parameters -->
-        <xacro:property name="base_mass" value="1.0" />
-        <xacro:property name="link0_mass" value="40.7" />
+        <xacro:property name="base_mass" value="44" />
+        <xacro:property name="link0_mass" value="7" />
         <xacro:property name="link1_mass" value="3.7" />
-        <xacro:property name="link2_mass" value="10.89" />
-        <xacro:property name="link3_mass" value="2.63" />
-        <xacro:property name="link4_mass" value="7.04" />
+        <xacro:property name="link2_mass" value="10.45" />
+        <xacro:property name="link3_mass" value="3.51" />
+        <xacro:property name="link4_mass" value="6.16" />
         <xacro:property name="link5_mass" value="0.87" />
-        <xacro:property name="link6_mass" value="0.44" />
+        <xacro:property name="link6_mass" value="0.88" />
         <xacro:property name="link1_radius" value="0.049" />
         <xacro:property name="link2_radius" value="0.045" />
@@ -103,6 +103,6 @@
         </link>
 <xacro:property name="joint1_type" value="revolute"/>
-<xacro:property name="joint1_axe" value="0 0 1"/>
-<xacro:property name="link1_length" value="0.42"/>
+<xacro:property name="joint1_axe" value="0 1 0"/>
+<xacro:property name="link1_length" value="0.1"/>
 <!--  joint 1    -->
         <joint name="${prefix}joint1" type="${joint1_type}">
@@ -134,10 +134,10 @@
 <xacro:property name="joint2_type" value="revolute"/>
 <xacro:property name="joint2_axe" value="0 1 0"/>
-<xacro:property name="link2_length" value="0.75"/>
+<xacro:property name="link2_length" value="0.7"/>
 <!--  joint 2   -->
         <joint name="${prefix}joint2" type="${joint2_type}">
           <parent link="${prefix}link1"/>
           <child link="${prefix}link2" />
-          <origin xyz="0 ${link1_radius+link2_radius} ${link1_length}" rpy="0 0 0 "/>
+          <origin xyz="0 0 ${link1_length + link2_radius}" rpy="${-1/2*pi} 0 0 "/>
           <axis xyz="${joint2_axe}"/>
           <xacro:joint_limit joint_type="${joint2_type}" link_length="${link2_length}"/>
@@ -164,5 +164,5 @@
 <xacro:property name="joint3_type" value="revolute"/>
 <xacro:property name="joint3_axe" value="0 1 0"/>
-<xacro:property name="link3_length" value="0.3"/>
+<xacro:property name="link3_length" value="0.4"/>
 <!--  joint 3   -->
         <joint name="${prefix}joint3" type="${joint3_type}">
@@ -194,10 +194,10 @@
 <xacro:property name="joint4_type" value="revolute"/>
 <xacro:property name="joint4_axe" value="0 1 0"/>
-<xacro:property name="link4_length" value="0.8"/>
+<xacro:property name="link4_length" value="0.7"/>
 <!--  joint 4   -->
         <joint name="${prefix}joint4" type="${joint4_type}">
           <parent link="${prefix}link3"/>
           <child link="${prefix}link4" />
-          <origin xyz="0 ${link3_radius+link4_radius} ${link3_length}" rpy="0 0 0 "/>
+          <origin xyz=" ${link3_radius+link4_radius} 0 ${link3_length}" rpy="0 0 ${-pi/2} "/>
           <axis xyz="${joint4_axe}"/>
           <xacro:joint_limit joint_type="${joint4_type}" link_length="${link4_length}"/>
@@ -254,5 +254,5 @@
 <xacro:property name="joint6_type" value="revolute"/>
 <xacro:property name="joint6_axe" value="0 1 0"/>
-<xacro:property name="link6_length" value="0.05"/>
+<xacro:property name="link6_length" value="0.1"/>
 <!--  joint 6   -->
         <joint name="${prefix}joint6" type="${joint6_type}">

File: man_gazebo/urdf/6dof/roll_z_0_1pitch_z_0_7pitch_y_0_4pitch_x_0_7roll_z_0_1pitch_y_0_11.urdf.xacro (robot description, xacro)
@@ -39,9 +39,9 @@
         <xacro:property name="link0_mass" value="40.7" />
         <xacro:property name="link1_mass" value="3.7" />
-        <xacro:property name="link2_mass" value="10.89" />
-        <xacro:property name="link3_mass" value="2.63" />
-        <xacro:property name="link4_mass" value="7.04" />
+        <xacro:property name="link2_mass" value="10.45" />
+        <xacro:property name="link3_mass" value="3.51" />
+        <xacro:property name="link4_mass" value="6.16" />
         <xacro:property name="link5_mass" value="0.87" />
-        <xacro:property name="link6_mass" value="0.44" />
+        <xacro:property name="link6_mass" value="0.97" />
         <xacro:property name="link1_radius" value="0.049" />
         <xacro:property name="link2_radius" value="0.045" />
@@ -103,6 +103,6 @@
         </link>
 <xacro:property name="joint1_type" value="revolute"/>
-<xacro:property name="joint1_axe" value="0 1 0"/>
-<xacro:property name="link1_length" value="0.44"/>
+<xacro:property name="joint1_axe" value="0 0 1"/>
+<xacro:property name="link1_length" value="0.1"/>
 <!--  joint 1    -->
         <joint name="${prefix}joint1" type="${joint1_type}">
@@ -134,10 +134,10 @@
 <xacro:property name="joint2_type" value="revolute"/>
 <xacro:property name="joint2_axe" value="0 1 0"/>
-<xacro:property name="link2_length" value="0.75"/>
+<xacro:property name="link2_length" value="0.7"/>
 <!--  joint 2   -->
         <joint name="${prefix}joint2" type="${joint2_type}">
           <parent link="${prefix}link1"/>
           <child link="${prefix}link2" />
-          <origin xyz="0 0 ${link1_length + link2_radius}" rpy="${-1/2*pi} 0 0 "/>
+          <origin xyz="0 0 ${link1_length + link2_radius}" rpy="${1/2*pi} 0 0 "/>
           <axis xyz="${joint2_axe}"/>
           <xacro:joint_limit joint_type="${joint2_type}" link_length="${link2_length}"/>
@@ -164,5 +164,5 @@
 <xacro:property name="joint3_type" value="revolute"/>
 <xacro:property name="joint3_axe" value="0 1 0"/>
-<xacro:property name="link3_length" value="0.3"/>
+<xacro:property name="link3_length" value="0.4"/>
 <!--  joint 3   -->
         <joint name="${prefix}joint3" type="${joint3_type}">
@@ -194,5 +194,5 @@
 <xacro:property name="joint4_type" value="revolute"/>
 <xacro:property name="joint4_axe" value="0 1 0"/>
-<xacro:property name="link4_length" value="0.8"/>
+<xacro:property name="link4_length" value="0.7"/>
 <!--  joint 4   -->
         <joint name="${prefix}joint4" type="${joint4_type}">
@@ -254,5 +254,5 @@
 <xacro:property name="joint6_type" value="revolute"/>
 <xacro:property name="joint6_axe" value="0 1 0"/>
-<xacro:property name="link6_length" value="0.05"/>
+<xacro:property name="link6_length" value="0.11"/>
 <!--  joint 6   -->
         <joint name="${prefix}joint6" type="${joint6_type}">

File: man_gazebo/urdf/6dofroll_z_0_1pitch_z_0_7pitch_y_0_4pitch_x_0_7roll_z_0_1pitch_y_0_11.urdf.xacro (robot description, xacro)
@@ -39,9 +39,9 @@
         <xacro:property name="link0_mass" value="40.7" />
         <xacro:property name="link1_mass" value="3.7" />
-        <xacro:property name="link2_mass" value="10.89" />
-        <xacro:property name="link3_mass" value="2.63" />
-        <xacro:property name="link4_mass" value="7.04" />
+        <xacro:property name="link2_mass" value="10.45" />
+        <xacro:property name="link3_mass" value="3.51" />
+        <xacro:property name="link4_mass" value="6.16" />
         <xacro:property name="link5_mass" value="0.87" />
-        <xacro:property name="link6_mass" value="0.44" />
+        <xacro:property name="link6_mass" value="0.97" />
         <xacro:property name="link1_radius" value="0.049" />
         <xacro:property name="link2_radius" value="0.045" />
@@ -104,5 +104,5 @@
 <xacro:property name="joint1_type" value="revolute"/>
 <xacro:property name="joint1_axe" value="0 0 1"/>
-<xacro:property name="link1_length" value="0.43"/>
+<xacro:property name="link1_length" value="0.1"/>
 <!--  joint 1    -->
         <joint name="${prefix}joint1" type="${joint1_type}">
@@ -133,11 +133,11 @@
         </link>
 <xacro:property name="joint2_type" value="revolute"/>
-<xacro:property name="joint2_axe" value="0 0 1"/>
-<xacro:property name="link2_length" value="0.75"/>
+<xacro:property name="joint2_axe" value="0 1 0"/>
+<xacro:property name="link2_length" value="0.7"/>
 <!--  joint 2   -->
         <joint name="${prefix}joint2" type="${joint2_type}">
           <parent link="${prefix}link1"/>
           <child link="${prefix}link2" />
-          <origin xyz="0 0 ${link2_radius + link1_length}" rpy="0 ${pi/2} 0 "/>
+          <origin xyz="0 0 ${link1_length + link2_radius}" rpy="${1/2*pi} 0 0 "/>
           <axis xyz="${joint2_axe}"/>
           <xacro:joint_limit joint_type="${joint2_type}" link_length="${link2_length}"/>
@@ -162,12 +162,12 @@
           </xacro:cylinder_inertial>
         </link>
-<xacro:property name="joint3_type" value="prismatic"/>
-<xacro:property name="joint3_axe" value="0 0 1"/>
-<xacro:property name="link3_length" value="0.3"/>
+<xacro:property name="joint3_type" value="revolute"/>
+<xacro:property name="joint3_axe" value="0 1 0"/>
+<xacro:property name="link3_length" value="0.4"/>
 <!--  joint 3   -->
         <joint name="${prefix}joint3" type="${joint3_type}">
           <parent link="${prefix}link2"/>
           <child link="${prefix}link3" />
-          <origin xyz="0 0 ${link2_length}" rpy="0 0 0 "/>
+          <origin xyz="0 ${link2_radius+link3_radius} ${link2_length}" rpy="0 0 0 "/>
           <axis xyz="${joint3_axe}"/>
           <xacro:joint_limit joint_type="${joint3_type}" link_length="${link3_length}"/>
@@ -194,10 +194,10 @@
 <xacro:property name="joint4_type" value="revolute"/>
 <xacro:property name="joint4_axe" value="0 1 0"/>
-<xacro:property name="link4_length" value="0.8"/>
+<xacro:property name="link4_length" value="0.7"/>
 <!--  joint 4   -->
         <joint name="${prefix}joint4" type="${joint4_type}">
           <parent link="${prefix}link3"/>
           <child link="${prefix}link4" />
-          <origin xyz="0 ${link3_radius+link4_radius} ${link3_length}" rpy="0 0 0 "/>
+          <origin xyz=" ${link3_radius+link4_radius} 0 ${link3_length}" rpy="0 0 ${-pi/2} "/>
           <axis xyz="${joint4_axe}"/>
           <xacro:joint_limit joint_type="${joint4_type}" link_length="${link4_length}"/>
@@ -254,5 +254,5 @@
 <xacro:property name="joint6_type" value="revolute"/>
 <xacro:property name="joint6_axe" value="0 1 0"/>
-<xacro:property name="link6_length" value="0.05"/>
+<xacro:property name="link6_length" value="0.11"/>
 <!--  joint 6   -->
         <joint name="${prefix}joint6" type="${joint6_type}">
