Commit message: working simulation process

File: man_gazebo/urdf/6dof/arms/_roll_y_0_1_pitch_x_0_7_pitch_y_0_6_pitch_y_0_7_pitch_y_0_2_roll_z_0_1.urdf.xacro (robot description, xacro)
@@ -32,16 +32,17 @@
         <xacro:macro name="arm_robot" params="prefix ">
         <xacro:property name="base_radius" value="0.060" />
+        <xacro:property name="base_length"  value="11" />
+        <xacro:property name="base_height"  value="1" />
+        <xacro:property name="base_width"  value="0.5" />
+        <xacro:property name="base_mass" value="44" />
+            <!-- Inertia parameters -->
+        <xacro:property name="link0_mass" value="7" />
+        <xacro:property name="link1_mass" value="3.7" />
+        <xacro:property name="link2_mass" value="5.12043" />
+        <xacro:property name="link3_mass" value="4.38894" />
+        <xacro:property name="link4_mass" value="5.12043" />
+        <xacro:property name="link5_mass" value="1.46298" />
+        <xacro:property name="link6_mass" value="0.73149" />
         <xacro:property name="link0_radius" value="0.060" />
-        <xacro:property name="base_length"  value="11" />
-        <xacro:property name="base_height"  value="0.5" />
-            <!-- Inertia parameters -->
-        <xacro:property name="base_mass" value="1.0" />
-        <xacro:property name="link0_mass" value="40.7" />
-        <xacro:property name="link1_mass" value="3.7" />
-        <xacro:property name="link2_mass" value="5.17" />
-        <xacro:property name="link3_mass" value="0.88" />
-        <xacro:property name="link4_mass" value="0.88" />
-        <xacro:property name="link5_mass" value="4.4" />
-        <xacro:property name="link6_mass" value="6.15" />
         <xacro:property name="link1_radius" value="0.049" />
         <xacro:property name="link2_radius" value="0.045" />
@@ -55,5 +56,5 @@
                 <origin xyz="0 0 ${base_height/2}" rpy="0 0 0" />
             <geometry>
-                    <box size="${base_height} ${base_length} ${base_height}"/>
+                    <box size="${base_width} ${base_length} ${base_height}"/>
             </geometry>
           </visual>
@@ -61,5 +62,5 @@
                  <origin xyz="0 0 ${base_height/2}" rpy="0 0 0" />
             <geometry>
-                    <box size="${base_length} ${base_length} ${base_height}"/>
+                    <box size="${base_width} ${base_length} ${base_height}"/>
             </geometry>
           </collision>
@@ -132,12 +133,12 @@
           </xacro:cylinder_inertial>
         </link>
-<xacro:property name="joint2_type" value="prismatic"/>
-<xacro:property name="joint2_axe" value="0 0 1"/>
-<xacro:property name="link2_length" value="0.1"/>
+<xacro:property name="joint2_type" value="revolute"/>
+<xacro:property name="joint2_axe" value="0 1 0"/>
+<xacro:property name="link2_length" value="0.7"/>
 <!--  joint 2   -->
         <joint name="${prefix}joint2" type="${joint2_type}">
           <parent link="${prefix}link1"/>
           <child link="${prefix}link2" />
-          <origin xyz="0 0 ${link1_length}" rpy="0 0 0 "/>
+          <origin xyz=" ${link1_radius+link2_radius} 0 ${link1_length}" rpy="0 0 ${-pi/2} "/>
           <axis xyz="${joint2_axe}"/>
           <xacro:joint_limit joint_type="${joint2_type}" link_length="${link2_length}"/>
@@ -163,11 +164,11 @@
         </link>
 <xacro:property name="joint3_type" value="revolute"/>
-<xacro:property name="joint3_axe" value="0 0 1"/>
-<xacro:property name="link3_length" value="0.1"/>
+<xacro:property name="joint3_axe" value="0 1 0"/>
+<xacro:property name="link3_length" value="0.6"/>
 <!--  joint 3   -->
         <joint name="${prefix}joint3" type="${joint3_type}">
           <parent link="${prefix}link2"/>
           <child link="${prefix}link3" />
-          <origin xyz="0 ${link2_radius} ${link2_length}" rpy="${-1/2*pi} 0 0 "/>
+          <origin xyz="0 ${link2_radius+link3_radius} ${link2_length}" rpy="0 0 0 "/>
           <axis xyz="${joint3_axe}"/>
           <xacro:joint_limit joint_type="${joint3_type}" link_length="${link3_length}"/>
@@ -193,11 +194,11 @@
         </link>
 <xacro:property name="joint4_type" value="revolute"/>
-<xacro:property name="joint4_axe" value="0 0 1"/>
-<xacro:property name="link4_length" value="0.1"/>
+<xacro:property name="joint4_axe" value="0 1 0"/>
+<xacro:property name="link4_length" value="0.7"/>
 <!--  joint 4   -->
         <joint name="${prefix}joint4" type="${joint4_type}">
           <parent link="${prefix}link3"/>
           <child link="${prefix}link4" />
-          <origin xyz="0 -${link3_radius} ${link3_length}" rpy="${1/2*pi} 0 0 "/>
+          <origin xyz="0 ${link3_radius+link4_radius} ${link3_length}" rpy="0 0 0 "/>
           <axis xyz="${joint4_axe}"/>
           <xacro:joint_limit joint_type="${joint4_type}" link_length="${link4_length}"/>
@@ -223,11 +224,11 @@
         </link>
 <xacro:property name="joint5_type" value="revolute"/>
-<xacro:property name="joint5_axe" value="0 0 1"/>
-<xacro:property name="link5_length" value="0.5"/>
+<xacro:property name="joint5_axe" value="0 1 0"/>
+<xacro:property name="link5_length" value="0.2"/>
 <!--  joint 5   -->
         <joint name="${prefix}joint5" type="${joint5_type}">
           <parent link="${prefix}link4"/>
           <child link="${prefix}link5" />
-          <origin xyz="0 ${link4_radius} ${link4_length}" rpy="${-1/2*pi} 0 0 "/>
+          <origin xyz="0 ${link4_radius+link5_radius} ${link4_length}" rpy="0 0 0 "/>
           <axis xyz="${joint5_axe}"/>
           <xacro:joint_limit joint_type="${joint5_type}" link_length="${link5_length}"/>
@@ -254,10 +255,10 @@
 <xacro:property name="joint6_type" value="revolute"/>
 <xacro:property name="joint6_axe" value="0 0 1"/>
-<xacro:property name="link6_length" value="0.7"/>
+<xacro:property name="link6_length" value="0.1"/>
 <!--  joint 6   -->
         <joint name="${prefix}joint6" type="${joint6_type}">
           <parent link="${prefix}link5"/>
           <child link="${prefix}link6" />
-          <origin xyz="0 -${link5_radius} ${link5_length}" rpy="${1/2*pi} 0 0 "/>
+          <origin xyz="0 0 ${link5_length}" rpy="0 0 0 "/>
           <axis xyz="${joint6_axe}"/>
           <xacro:joint_limit joint_type="${joint6_type}" link_length="${link6_length}"/>
@@ -282,8 +283,8 @@
           </xacro:cylinder_inertial>
         </link>
-        <!-- camera joint - fictive joint -->
-        <joint name="camera_joint" type="revolute">
+        <!-- Sprayer joint - fictive joint -->
+        <joint name="sprayer_joint" type="revolute">
             <parent link="${prefix}link6" />
-            <child link = "camera_link" />
+            <child link = "sprayer_link" />
             <origin xyz="0.0  0.0 ${link6_length}" rpy="0.0 0.0 0" />
             <axis xyz="0 0 1"/>
@@ -291,6 +292,6 @@
             <dynamics damping="0.0" friction="0.0"/>
         </joint>
-        <!-- Camera -->
-        <link name="camera_link">
+        <!-- Sprayer -->
+        <link name="sprayer_link">
           <collision>
             <origin rpy="0 0 0" xyz="0 0 0.005"/>
@@ -319,5 +320,5 @@
             <!-- ee joint -->
         <joint name="${prefix}ee_fixed_joint" type="fixed">
-          <parent link="camera_link" />
+          <parent link="sprayer_link" />
           <child link = "${prefix}ee_link" />
           <origin xyz="0.0  0.0 0.01" rpy="0.0 0.0 0" />

File: man_gazebo/urdf/6dof/manipulator.urdf.xacro (robot description, xacro)
@@ -48,5 +48,6 @@
 	<xacro:property name="link0_length" value="0.25" />
  	<xacro:property name="base_length"  value="11" />
-  	<xacro:property name="base_height"  value="0.5" />
+  <xacro:property name="base_height"  value="1" />
+  <xacro:property name="base_width"  value="0.5" />
 	<xacro:property name="link1_length" value="0.25" />
 	<xacro:property name="link2_length" value="0.5" />
@@ -65,5 +66,5 @@
     <xacro:property name="link6_mass" value="0.1879" />
     <xacro:property name="base_radius" value="0.060" />
-	<xacro:property name="link0_radius" value="0.060" />
+	  <xacro:property name="link0_radius" value="0.060" />
     <xacro:property name="link1_radius" value="0.060" />
     <xacro:property name="link2_radius" value="0.060" />
@@ -77,5 +78,5 @@
 		    <origin xyz="0 0 ${base_height/2}" rpy="0 0 0" />
         <geometry>
- 			    <box size="${base_height} ${base_length} ${base_height}"/>
+ 			    <box size="${base_width} ${base_length} ${base_height}"/>
         </geometry>
       </visual>
@@ -83,5 +84,5 @@
 			 <origin xyz="0 0 ${base_height/2}" rpy="0 0 0" />
         <geometry>
-			    <box size="${base_length} ${base_length} ${base_height}"/>
+			    <box size="${base_width} ${base_length} ${base_height}"/>
         </geometry>
       </collision>

File: man_gazebo/urdf/gazebo.xacro (robot description, xacro)
@@ -51,5 +51,5 @@
       <selfCollide>true</selfCollide>
     </gazebo>
-    <gazebo reference="camera_link">
+    <gazebo reference="sprayer_link">
       <selfCollide>true</selfCollide>
     </gazebo>
