Commit message: not working

File: man_gazebo/urdf/6dof/arms/arm.urdf.xacro (robot description, xacro)
@@ -41,5 +41,6 @@
         <xacro:property name="joint6_axe" value="0 0 1" />
         <xacro:property name="base_length"  value="11" />
-        <xacro:property name="base_height"  value="0.5" />
+        <xacro:property name="base_height"  value="1" />
+	<xacro:property name="base_width"  value="0.5" />
         <xacro:property name="link0_length" value="0.25" />
         <xacro:property name="link1_length" value="0.75" />
@@ -79,5 +80,5 @@
 		    <origin xyz="0 0 ${base_height/2}" rpy="0 0 0" />
         <geometry>
- 			    <box size="${base_height} ${base_length} ${base_height}"/>
+ 			    <box size="${base_width} ${base_length} ${base_height}"/>
         </geometry>
       </visual>
@@ -85,5 +86,5 @@
 			 <origin xyz="0 0 ${base_height/2}" rpy="0 0 0" />
         <geometry>
-			    <box size="${base_length} ${base_length} ${base_height}"/>
+			    <box size="${base_width} ${base_length} ${base_height}"/>
         </geometry>
       </collision>

File: man_gazebo/urdf/6dof/arms/manipulator.urdf.xacro (robot description, xacro)
@@ -48,6 +48,6 @@
 	<xacro:property name="link0_length" value="0.25" />
  	<xacro:property name="base_length"  value="11" />
-  <xacro:property name="base_height"  value="1" />
-  <xacro:property name="base_width"  value="0.5" />
+	 <xacro:property name="base_height"  value="1" />
+	 <xacro:property name="base_width"  value="0.5" />
 	<xacro:property name="link1_length" value="0.25" />
 	<xacro:property name="link2_length" value="0.5" />
