Commit message: g

File: man_gazebo/urdf/4dof/_roll_z_0_1_roll_y_0_5_roll_y_0_3_pitch_y_0_5_pitch_y_0_3_pitch_y_0_1.urdf.xacro (robot description, xacro)
@@ -5,4 +5,10 @@
         <xacro:include filename="$(find man_gazebo)/urdf/gazebo.xacro" />
         <xacro:macro name="cylinder_inertial" params="radius length mass *origin">
+        <link name="world" />
+          <joint name="world_joint" type="fixed">
+            <parent link="world" />
+            <child link = "base_link" />
+            <origin xyz="0 0 0" rpy="0.0 0.0 0.0" />
+          </joint>
         <inertial>
           <mass value="${mass}" />
@@ -33,5 +39,5 @@
         <xacro:property name="link0_mass" value="7" />
         <xacro:property name="link1_mass" value="3.7" />
-        <xacro:property name="link2_mass" value="5.12043" />
+        <xacro:property name="link2_mass" value="3.65745" />
         <xacro:property name="link3_mass" value="2.19447" />
         <xacro:property name="link4_mass" value="3.65745" />
@@ -45,10 +51,4 @@
         <xacro:property name="link5_radius" value="0.030" />
         <xacro:property name="link6_radius" value="0.025" />
-        <link name="world" />
-          <joint name="world_joint" type="fixed">
-            <parent link="world" />
-            <child link = "base_link" />
-            <origin xyz="0 0 0" rpy="0.0 0.0 0.0" />
-          </joint>
         <!-- Base Link -->
         <link name="${prefix}base_link" >
@@ -133,12 +133,12 @@
           </xacro:cylinder_inertial>
         </link>
-<xacro:property name="joint2_type" value="prismatic"/>
+<xacro:property name="joint2_type" value="revolute"/>
 <xacro:property name="joint2_axe" value="0 0 1"/>
-<xacro:property name="link2_length" value="0.7"/>
+<xacro:property name="link2_length" value="0.5"/>
 <!--  joint 2   -->
         <joint name="${prefix}joint2" type="${joint2_type}">
           <parent link="${prefix}link1"/>
           <child link="${prefix}link2" />
-          <origin xyz="0 0 ${link1_length}" rpy="0 0 0 "/>
+          <origin xyz="0 ${link1_radius} ${link1_length}" rpy="${-1/2*pi} 0 0 "/>
           <axis xyz="${joint2_axe}"/>
           <xacro:joint_limit joint_type="${joint2_type}" link_length="${link2_length}"/>
@@ -170,5 +170,5 @@
           <parent link="${prefix}link2"/>
           <child link="${prefix}link3" />
-          <origin xyz="0 ${link2_radius} ${link2_length}" rpy="${-1/2*pi} 0 0 "/>
+          <origin xyz="0 -${link2_radius} ${link2_length}" rpy="${1/2*pi} 0 0 "/>
           <axis xyz="${joint3_axe}"/>
           <xacro:joint_limit joint_type="${joint3_type}" link_length="${link3_length}"/>
@@ -194,5 +194,5 @@
         </link>
 <xacro:property name="joint4_type" value="revolute"/>
-<xacro:property name="joint4_axe" value="0 0 1"/>
+<xacro:property name="joint4_axe" value="0 1 0"/>
 <xacro:property name="link4_length" value="0.5"/>
 <!--  joint 4   -->
@@ -200,5 +200,5 @@
           <parent link="${prefix}link3"/>
           <child link="${prefix}link4" />
-          <origin xyz="0 -${link3_radius} ${link3_length}" rpy="${1/2*pi} 0 0 "/>
+          <origin xyz="0 ${link3_radius+link4_radius} ${link3_length}" rpy="0 0 0 "/>
           <axis xyz="${joint4_axe}"/>
           <xacro:joint_limit joint_type="${joint4_type}" link_length="${link4_length}"/>
@@ -223,17 +223,17 @@
           </xacro:cylinder_inertial>
         </link>
-<xacro:property name="joint5_type" value="revolute"/>
-<xacro:property name="joint5_axe" value="0 0 1"/>
+<!--<xacro:property name="joint5_type" value="revolute"/>
+<xacro:property name="joint5_axe" value="0 1 0"/>
 <xacro:property name="link5_length" value="0.3"/>
-<!--  joint 5   -->
+  joint 5
         <joint name="${prefix}joint5" type="${joint5_type}">
           <parent link="${prefix}link4"/>
           <child link="${prefix}link5" />
-          <origin xyz="0 ${link4_radius} ${link4_length}" rpy="${-1/2*pi} 0 0 "/>
+          <origin xyz="0 ${link4_radius+link5_radius} ${link4_length}" rpy="0 0 0 "/>
           <axis xyz="${joint5_axe}"/>
           <xacro:joint_limit joint_type="${joint5_type}" link_length="${link5_length}"/>
           <dynamics damping="0.0" friction="0.0"/>
-        </joint>
-    <!-- link 5   -->
+        </joint>-->
+    <!-- link 5
         <link name="${prefix}link5">
           <visual>
@@ -252,18 +252,18 @@
             <origin xyz="0.0 0.0 ${link5_length / 2 }" rpy="0 0 0" />
           </xacro:cylinder_inertial>
-        </link>
-<xacro:property name="joint6_type" value="prismatic"/>
-<xacro:property name="joint6_axe" value="0 0 1"/>
+        </link> -->
+<!--<xacro:property name="joint6_type" value="revolute"/>
+<xacro:property name="joint6_axe" value="0 1 0"/>
 <xacro:property name="link6_length" value="0.1"/>
-<!--  joint 6   -->
+  joint 6
         <joint name="${prefix}joint6" type="${joint6_type}">
           <parent link="${prefix}link5"/>
           <child link="${prefix}link6" />
-          <origin xyz="0 0 ${link5_length + link6_radius}" rpy="${-1/2*pi} 0 0 "/>
+          <origin xyz="0 ${link5_radius+link6_radius} ${link5_length}" rpy="0 0 0 "/>
           <axis xyz="${joint6_axe}"/>
           <xacro:joint_limit joint_type="${joint6_type}" link_length="${link6_length}"/>
           <dynamics damping="0.0" friction="0.0"/>
-        </joint>
-    <!-- link 6   -->
+        </joint>  -->
+    <!-- link 6
         <link name="${prefix}link6">
           <visual>
@@ -282,10 +282,10 @@
             <origin xyz="0.0 0.0 ${link6_length / 2 }" rpy="0 0 0" />
           </xacro:cylinder_inertial>
-        </link>
+        </link>-->
         <!-- Sprayer joint - fictive joint -->
         <joint name="fake_joint" type="revolute">
-            <parent link="${prefix}link6" />
+            <parent link="${prefix}link4" />
             <child link = "camera_link" />
-            <origin xyz="0.0  0.0 ${link6_length}" rpy="0.0 0.0 0" />
+            <origin xyz="0.0  0.0 ${link4_length}" rpy="0.0 0.0 0" />
             <axis xyz="0 0 1"/>
             <xacro:joint_limit joint_type="revolute" link_length="0.1"/>

File: man_gazebo/urdf/4dof/_roll_z_0_1_roll_y_0_5_roll_y_0_5_pitch_y_0_3.urdf.xacro (robot description, xacro)
@@ -2,7 +2,13 @@
         <robot xmlns:xacro="http://wiki.ros.org/xacro"  name="arm">
         <xacro:include filename="$(find man_gazebo)/urdf/common.gazebo.xacro" />
-        <xacro:include filename="$(find man_gazebo)/urdf/6dof/transmission_6dof.xacro" />
+        <xacro:include filename="$(find man_gazebo)/urdf/4dof/transmission_4dof.xacro" />
         <xacro:include filename="$(find man_gazebo)/urdf/gazebo.xacro" />
         <xacro:macro name="cylinder_inertial" params="radius length mass *origin">
+        <link name="world" />
+          <joint name="world_joint" type="fixed">
+            <parent link="world" />
+            <child link = "base_link" />
+            <origin xyz="0 0 0" rpy="0.0 0.0 0.0" />
+          </joint>
         <inertial>
           <mass value="${mass}" />
@@ -33,9 +39,9 @@
         <xacro:property name="link0_mass" value="7" />
         <xacro:property name="link1_mass" value="3.7" />
-        <xacro:property name="link2_mass" value="5.12043" />
-        <xacro:property name="link3_mass" value="2.19447" />
-        <xacro:property name="link4_mass" value="3.65745" />
-        <xacro:property name="link5_mass" value="2.19447" />
-        <xacro:property name="link6_mass" value="0.73149" />
+        <xacro:property name="link2_mass" value="3.65745" />
+        <xacro:property name="link3_mass" value="3.65745" />
+        <xacro:property name="link4_mass" value="2.19447" />
+        <xacro:property name="link5_mass" value="0" />
+        <xacro:property name="link6_mass" value="0" />
         <xacro:property name="link0_radius" value="0.060" />
         <xacro:property name="link1_radius" value="0.049" />
@@ -45,10 +51,4 @@
         <xacro:property name="link5_radius" value="0.030" />
         <xacro:property name="link6_radius" value="0.025" />
-        <link name="world" />
-          <joint name="world_joint" type="fixed">
-            <parent link="world" />
-            <child link = "base_link" />
-            <origin xyz="0 0 0" rpy="0.0 0.0 0.0" />
-          </joint>
         <!-- Base Link -->
         <link name="${prefix}base_link" >
@@ -133,12 +133,12 @@
           </xacro:cylinder_inertial>
         </link>
-<xacro:property name="joint2_type" value="prismatic"/>
+<xacro:property name="joint2_type" value="revolute"/>
 <xacro:property name="joint2_axe" value="0 0 1"/>
-<xacro:property name="link2_length" value="0.7"/>
+<xacro:property name="link2_length" value="0.5"/>
 <!--  joint 2   -->
         <joint name="${prefix}joint2" type="${joint2_type}">
           <parent link="${prefix}link1"/>
           <child link="${prefix}link2" />
-          <origin xyz="0 0 ${link1_length}" rpy="0 0 0 "/>
+          <origin xyz="0 ${link1_radius} ${link1_length}" rpy="${-1/2*pi} 0 0 "/>
           <axis xyz="${joint2_axe}"/>
           <xacro:joint_limit joint_type="${joint2_type}" link_length="${link2_length}"/>
@@ -165,10 +165,10 @@
 <xacro:property name="joint3_type" value="revolute"/>
 <xacro:property name="joint3_axe" value="0 0 1"/>
-<xacro:property name="link3_length" value="0.3"/>
+<xacro:property name="link3_length" value="0.5"/>
 <!--  joint 3   -->
         <joint name="${prefix}joint3" type="${joint3_type}">
           <parent link="${prefix}link2"/>
           <child link="${prefix}link3" />
-          <origin xyz="0 ${link2_radius} ${link2_length}" rpy="${-1/2*pi} 0 0 "/>
+          <origin xyz="0 -${link2_radius} ${link2_length}" rpy="${1/2*pi} 0 0 "/>
           <axis xyz="${joint3_axe}"/>
           <xacro:joint_limit joint_type="${joint3_type}" link_length="${link3_length}"/>
@@ -194,11 +194,11 @@
         </link>
 <xacro:property name="joint4_type" value="revolute"/>
-<xacro:property name="joint4_axe" value="0 0 1"/>
-<xacro:property name="link4_length" value="0.5"/>
+<xacro:property name="joint4_axe" value="0 1 0"/>
+<xacro:property name="link4_length" value="0.3"/>
 <!--  joint 4   -->
         <joint name="${prefix}joint4" type="${joint4_type}">
           <parent link="${prefix}link3"/>
           <child link="${prefix}link4" />
-          <origin xyz="0 -${link3_radius} ${link3_length}" rpy="${1/2*pi} 0 0 "/>
+          <origin xyz="0 ${link3_radius+link4_radius} ${link3_length}" rpy="0 0 0 "/>
           <axis xyz="${joint4_axe}"/>
           <xacro:joint_limit joint_type="${joint4_type}" link_length="${link4_length}"/>
@@ -223,69 +223,9 @@
           </xacro:cylinder_inertial>
         </link>
-<xacro:property name="joint5_type" value="revolute"/>
-<xacro:property name="joint5_axe" value="0 0 1"/>
-<xacro:property name="link5_length" value="0.3"/>
-<!--  joint 5   -->
-        <joint name="${prefix}joint5" type="${joint5_type}">
-          <parent link="${prefix}link4"/>
-          <child link="${prefix}link5" />
-          <origin xyz="0 ${link4_radius} ${link4_length}" rpy="${-1/2*pi} 0 0 "/>
-          <axis xyz="${joint5_axe}"/>
-          <xacro:joint_limit joint_type="${joint5_type}" link_length="${link5_length}"/>
-          <dynamics damping="0.0" friction="0.0"/>
-        </joint>
-    <!-- link 5   -->
-        <link name="${prefix}link5">
-          <visual>
-            <origin xyz="0 0 ${link5_length / 2}" rpy="0 0 0" />
-            <geometry>
-                <cylinder radius="${link5_radius}" length="${link5_length}"/>
-            </geometry>
-          </visual>
-          <collision>
-            <origin xyz="0 0 ${link5_length / 2 }" rpy="0 0 0" />
-            <geometry>
-                <cylinder radius="${link5_radius}" length="${link5_length}"/>
-            </geometry>
-          </collision>
-          <xacro:cylinder_inertial radius="${link5_radius}" length="${link5_length}" mass="${link5_mass}">
-            <origin xyz="0.0 0.0 ${link5_length / 2 }" rpy="0 0 0" />
-          </xacro:cylinder_inertial>
-        </link>
-<xacro:property name="joint6_type" value="prismatic"/>
-<xacro:property name="joint6_axe" value="0 0 1"/>
-<xacro:property name="link6_length" value="0.1"/>
-<!--  joint 6   -->
-        <joint name="${prefix}joint6" type="${joint6_type}">
-          <parent link="${prefix}link5"/>
-          <child link="${prefix}link6" />
-          <origin xyz="0 0 ${link5_length + link6_radius}" rpy="${-1/2*pi} 0 0 "/>
-          <axis xyz="${joint6_axe}"/>
-          <xacro:joint_limit joint_type="${joint6_type}" link_length="${link6_length}"/>
-          <dynamics damping="0.0" friction="0.0"/>
-        </joint>
-    <!-- link 6   -->
-        <link name="${prefix}link6">
-          <visual>
-            <origin xyz="0 0 ${link6_length / 2}" rpy="0 0 0" />
-            <geometry>
-                <cylinder radius="${link6_radius}" length="${link6_length}"/>
-            </geometry>
-          </visual>
-          <collision>
-            <origin xyz="0 0 ${link6_length / 2 }" rpy="0 0 0" />
-            <geometry>
-                <cylinder radius="${link6_radius}" length="${link6_length}"/>
-            </geometry>
-          </collision>
-          <xacro:cylinder_inertial radius="${link6_radius}" length="${link6_length}" mass="${link6_mass}">
-            <origin xyz="0.0 0.0 ${link6_length / 2 }" rpy="0 0 0" />
-          </xacro:cylinder_inertial>
-        </link>
         <!-- Sprayer joint - fictive joint -->
         <joint name="fake_joint" type="revolute">
-            <parent link="${prefix}link6" />
+            <parent link="${prefix}link4" />
             <child link = "camera_link" />
-            <origin xyz="0.0  0.0 ${link6_length}" rpy="0.0 0.0 0" />
+            <origin xyz="0.0  0.0 ${link4_length}" rpy="0.0 0.0 0" />
             <axis xyz="0 0 1"/>
             <xacro:joint_limit joint_type="revolute" link_length="0.1"/>

File: man_gazebo/urdf/5dof/_roll_z_0_1_pitch_z_0_3_pitch_y_0_3_pris_z_0_5_pris_x_0_5_pris_z_0_1.urdf.xacro (robot description, xacro)
@@ -39,8 +39,8 @@
         <xacro:property name="link0_mass" value="7" />
         <xacro:property name="link1_mass" value="3.7" />
-        <xacro:property name="link2_mass" value="3.65745" />
-        <xacro:property name="link3_mass" value="3.65745" />
-        <xacro:property name="link4_mass" value="2.19447" />
-        <xacro:property name="link5_mass" value="0.73149" />
+        <xacro:property name="link2_mass" value="2.19447" />
+        <xacro:property name="link3_mass" value="2.19447" />
+        <xacro:property name="link4_mass" value="3.65745" />
+        <xacro:property name="link5_mass" value="3.65745" />
         <xacro:property name="link6_mass" value="0.73149" />
         <xacro:property name="link0_radius" value="0.060" />
@@ -133,12 +133,12 @@
           </xacro:cylinder_inertial>
         </link>
-<xacro:property name="joint2_type" value="prismatic"/>
-<xacro:property name="joint2_axe" value="0 0 1"/>
-<xacro:property name="link2_length" value="0.5"/>
+<xacro:property name="joint2_type" value="revolute"/>
+<xacro:property name="joint2_axe" value="0 1 0"/>
+<xacro:property name="link2_length" value="0.3"/>
 <!--  joint 2   -->
         <joint name="${prefix}joint2" type="${joint2_type}">
           <parent link="${prefix}link1"/>
           <child link="${prefix}link2" />
-          <origin xyz="0 0 ${link1_length}" rpy="0 0 0 "/>
+          <origin xyz="0 0 ${link1_length + link2_radius}" rpy="${1/2*pi} 0 0 "/>
           <axis xyz="${joint2_axe}"/>
           <xacro:joint_limit joint_type="${joint2_type}" link_length="${link2_length}"/>
@@ -163,12 +163,12 @@
           </xacro:cylinder_inertial>
         </link>
-<xacro:property name="joint3_type" value="prismatic"/>
-<xacro:property name="joint3_axe" value="0 0 1"/>
-<xacro:property name="link3_length" value="0.5"/>
+<xacro:property name="joint3_type" value="revolute"/>
+<xacro:property name="joint3_axe" value="0 1 0"/>
+<xacro:property name="link3_length" value="0.3"/>
 <!--  joint 3   -->
         <joint name="${prefix}joint3" type="${joint3_type}">
           <parent link="${prefix}link2"/>
           <child link="${prefix}link3" />
-          <origin xyz="0 0 ${link2_length + link3_radius}" rpy="${-1/2*pi} 0 0 "/>
+          <origin xyz="0 ${link2_radius+link3_radius} ${link2_length}" rpy="0 0 0 "/>
           <axis xyz="${joint3_axe}"/>
           <xacro:joint_limit joint_type="${joint3_type}" link_length="${link3_length}"/>
@@ -193,12 +193,12 @@
           </xacro:cylinder_inertial>
         </link>
-<xacro:property name="joint4_type" value="revolute"/>
-<xacro:property name="joint4_axe" value="0 1 0"/>
-<xacro:property name="link4_length" value="0.3"/>
+<xacro:property name="joint4_type" value="prismatic"/>
+<xacro:property name="joint4_axe" value="0 0 1"/>
+<xacro:property name="link4_length" value="0.5"/>
 <!--  joint 4   -->
         <joint name="${prefix}joint4" type="${joint4_type}">
           <parent link="${prefix}link3"/>
           <child link="${prefix}link4" />
-          <origin xyz="0 0 ${link3_length + link4_radius}" rpy="${1/2*pi} 0 0 "/>
+          <origin xyz="0 0 ${link3_length}" rpy="0 0 0 "/>
           <axis xyz="${joint4_axe}"/>
           <xacro:joint_limit joint_type="${joint4_type}" link_length="${link4_length}"/>
@@ -223,12 +223,12 @@
           </xacro:cylinder_inertial>
         </link>
-<xacro:property name="joint5_type" value="revolute"/>
-<xacro:property name="joint5_axe" value="0 1 0"/>
-<xacro:property name="link5_length" value="0.1"/>
+<xacro:property name="joint5_type" value="prismatic"/>
+<xacro:property name="joint5_axe" value="0 0 1"/>
+<xacro:property name="link5_length" value="0.5"/>
 <!--  joint 5   -->
         <joint name="${prefix}joint5" type="${joint5_type}">
           <parent link="${prefix}link4"/>
           <child link="${prefix}link5" />
-          <origin xyz=" ${link4_radius+link5_radius} 0 ${link4_length}" rpy="0 0 ${-pi/2} "/>
+          <origin xyz="0 0 ${link4_length + link5_radius}" rpy="0 ${-pi/2} 0 "/>
           <axis xyz="${joint5_axe}"/>
           <xacro:joint_limit joint_type="${joint5_type}" link_length="${link5_length}"/>
@@ -253,8 +253,8 @@
           </xacro:cylinder_inertial>
         </link>
-<xacro:property name="joint6_type" value="revolute"/>
+<!--<xacro:property name="joint6_type" value="prismatic"/>
 <xacro:property name="joint6_axe" value="0 0 1"/>
 <xacro:property name="link6_length" value="0.1"/>
-<!--  joint 6   -->
+  joint 6
         <joint name="${prefix}joint6" type="${joint6_type}">
           <parent link="${prefix}link5"/>
@@ -264,6 +264,6 @@
           <xacro:joint_limit joint_type="${joint6_type}" link_length="${link6_length}"/>
           <dynamics damping="0.0" friction="0.0"/>
-        </joint>
-    <!-- link 6   -->
+        </joint>-->
+    <!-- link 6
         <link name="${prefix}link6">
           <visual>
@@ -282,10 +282,10 @@
             <origin xyz="0.0 0.0 ${link6_length / 2 }" rpy="0 0 0" />
           </xacro:cylinder_inertial>
-        </link>
+        </link> -->
         <!-- Sprayer joint - fictive joint -->
         <joint name="fake_joint" type="revolute">
-            <parent link="${prefix}link6" />
+            <parent link="${prefix}link5" />
             <child link = "camera_link" />
-            <origin xyz="0.0  0.0 ${link6_length}" rpy="0.0 0.0 0" />
+            <origin xyz="0.0  0.0 ${link5_length}" rpy="0.0 0.0 0" />
             <axis xyz="0 0 1"/>
             <xacro:joint_limit joint_type="revolute" link_length="0.1"/>
