Commit message: g

File: man_gazebo/urdf/5dof/_roll_z_0_1_roll_y_0_5_roll_y_0_3_pitch_y_0_3_pitch_y_0_3.urdf.xacro (robot description, xacro)
@@ -2,5 +2,5 @@
         <robot xmlns:xacro="http://wiki.ros.org/xacro"  name="arm">
         <xacro:include filename="$(find man_gazebo)/urdf/common.gazebo.xacro" />
-        <xacro:include filename="$(find man_gazebo)/urdf/6dof/transmission_6dof.xacro" />
+        <xacro:include filename="$(find man_gazebo)/urdf/5dof/transmission_5dof.xacro" />
         <xacro:include filename="$(find man_gazebo)/urdf/gazebo.xacro" />
         <xacro:macro name="cylinder_inertial" params="radius length mass *origin">
@@ -41,7 +41,7 @@
         <xacro:property name="link2_mass" value="3.65745" />
         <xacro:property name="link3_mass" value="2.19447" />
-        <xacro:property name="link4_mass" value="3.65745" />
+        <xacro:property name="link4_mass" value="2.19447" />
         <xacro:property name="link5_mass" value="2.19447" />
-        <xacro:property name="link6_mass" value="0.73149" />
+        <xacro:property name="link6_mass" value="0" />
         <xacro:property name="link0_radius" value="0.060" />
         <xacro:property name="link1_radius" value="0.049" />
@@ -133,5 +133,5 @@
           </xacro:cylinder_inertial>
         </link>
-<xacro:property name="joint2_type" value="prismatic"/>
+<xacro:property name="joint2_type" value="revolute"/>
 <xacro:property name="joint2_axe" value="0 0 1"/>
 <xacro:property name="link2_length" value="0.5"/>
@@ -140,5 +140,5 @@
           <parent link="${prefix}link1"/>
           <child link="${prefix}link2" />
-          <origin xyz="0 0 ${link1_length}" rpy="0 0 0 "/>
+          <origin xyz="0 ${link1_radius} ${link1_length}" rpy="${-1/2*pi} 0 0 "/>
           <axis xyz="${joint2_axe}"/>
           <xacro:joint_limit joint_type="${joint2_type}" link_length="${link2_length}"/>
@@ -170,5 +170,5 @@
           <parent link="${prefix}link2"/>
           <child link="${prefix}link3" />
-          <origin xyz="0 ${link2_radius} ${link2_length}" rpy="${-1/2*pi} 0 0 "/>
+          <origin xyz="0 -${link2_radius} ${link2_length}" rpy="${1/2*pi} 0 0 "/>
           <axis xyz="${joint3_axe}"/>
           <xacro:joint_limit joint_type="${joint3_type}" link_length="${link3_length}"/>
@@ -194,11 +194,11 @@
         </link>
 <xacro:property name="joint4_type" value="revolute"/>
-<xacro:property name="joint4_axe" value="0 0 1"/>
-<xacro:property name="link4_length" value="0.5"/>
+<xacro:property name="joint4_axe" value="0 1 0"/>
+<xacro:property name="link4_length" value="0.3"/>
 <!--  joint 4   -->
         <joint name="${prefix}joint4" type="${joint4_type}">
           <parent link="${prefix}link3"/>
           <child link="${prefix}link4" />
-          <origin xyz="0 -${link3_radius} ${link3_length}" rpy="${1/2*pi} 0 0 "/>
+          <origin xyz="0 ${link3_radius+link4_radius} ${link3_length}" rpy="0 0 0 "/>
           <axis xyz="${joint4_axe}"/>
           <xacro:joint_limit joint_type="${joint4_type}" link_length="${link4_length}"/>
@@ -224,5 +224,5 @@
         </link>
 <xacro:property name="joint5_type" value="revolute"/>
-<xacro:property name="joint5_axe" value="0 0 1"/>
+<xacro:property name="joint5_axe" value="0 1 0"/>
 <xacro:property name="link5_length" value="0.3"/>
 <!--  joint 5   -->
@@ -230,5 +230,5 @@
           <parent link="${prefix}link4"/>
           <child link="${prefix}link5" />
-          <origin xyz="0 ${link4_radius} ${link4_length}" rpy="${-1/2*pi} 0 0 "/>
+          <origin xyz="0 ${link4_radius+link5_radius} ${link4_length}" rpy="0 0 0 "/>
           <axis xyz="${joint5_axe}"/>
           <xacro:joint_limit joint_type="${joint5_type}" link_length="${link5_length}"/>
@@ -253,39 +253,9 @@
           </xacro:cylinder_inertial>
         </link>
-<xacro:property name="joint6_type" value="revolute"/>
-<xacro:property name="joint6_axe" value="0 1 0"/>
-<xacro:property name="link6_length" value="0.1"/>
-<!--  joint 6   -->
-        <joint name="${prefix}joint6" type="${joint6_type}">
-          <parent link="${prefix}link5"/>
-          <child link="${prefix}link6" />
-          <origin xyz="0 0 ${link5_length + link6_radius}" rpy="${1/2*pi} 0 0 "/>
-          <axis xyz="${joint6_axe}"/>
-          <xacro:joint_limit joint_type="${joint6_type}" link_length="${link6_length}"/>
-          <dynamics damping="0.0" friction="0.0"/>
-        </joint>
-    <!-- link 6   -->
-        <link name="${prefix}link6">
-          <visual>
-            <origin xyz="0 0 ${link6_length / 2}" rpy="0 0 0" />
-            <geometry>
-                <cylinder radius="${link6_radius}" length="${link6_length}"/>
-            </geometry>
-          </visual>
-          <collision>
-            <origin xyz="0 0 ${link6_length / 2 }" rpy="0 0 0" />
-            <geometry>
-                <cylinder radius="${link6_radius}" length="${link6_length}"/>
-            </geometry>
-          </collision>
-          <xacro:cylinder_inertial radius="${link6_radius}" length="${link6_length}" mass="${link6_mass}">
-            <origin xyz="0.0 0.0 ${link6_length / 2 }" rpy="0 0 0" />
-          </xacro:cylinder_inertial>
-        </link>
         <!-- Sprayer joint - fictive joint -->
         <joint name="fake_joint" type="revolute">
-            <parent link="${prefix}link6" />
+            <parent link="${prefix}link5" />
             <child link = "camera_link" />
-            <origin xyz="0.0  0.0 ${link6_length}" rpy="0.0 0.0 0" />
+            <origin xyz="0.0  0.0 ${link5_length}" rpy="0.0 0.0 0" />
             <axis xyz="0 0 1"/>
             <xacro:joint_limit joint_type="revolute" link_length="0.1"/>

File: man_gazebo/urdf/5dof/_roll_z_0_1_roll_y_0_5_roll_y_0_3_pitch_y_0_5_pitch_y_0_3_pitch_y_0_1.urdf.xacro (robot description, xacro)
@@ -5,4 +5,10 @@
         <xacro:include filename="$(find man_gazebo)/urdf/gazebo.xacro" />
         <xacro:macro name="cylinder_inertial" params="radius length mass *origin">
+        <link name="world" />
+          <joint name="world_joint" type="fixed">
+            <parent link="world" />
+            <child link = "base_link" />
+            <origin xyz="0 0 0" rpy="0.0 0.0 0.0" />
+          </joint>
         <inertial>
           <mass value="${mass}" />
@@ -33,5 +39,5 @@
         <xacro:property name="link0_mass" value="7" />
         <xacro:property name="link1_mass" value="3.7" />
-        <xacro:property name="link2_mass" value="5.12043" />
+        <xacro:property name="link2_mass" value="3.65745" />
         <xacro:property name="link3_mass" value="2.19447" />
         <xacro:property name="link4_mass" value="3.65745" />
@@ -45,10 +51,4 @@
         <xacro:property name="link5_radius" value="0.030" />
         <xacro:property name="link6_radius" value="0.025" />
-        <link name="world" />
-          <joint name="world_joint" type="fixed">
-            <parent link="world" />
-            <child link = "base_link" />
-            <origin xyz="0 0 0" rpy="0.0 0.0 0.0" />
-          </joint>
         <!-- Base Link -->
         <link name="${prefix}base_link" >
@@ -133,12 +133,12 @@
           </xacro:cylinder_inertial>
         </link>
-<xacro:property name="joint2_type" value="prismatic"/>
+<xacro:property name="joint2_type" value="revolute"/>
 <xacro:property name="joint2_axe" value="0 0 1"/>
-<xacro:property name="link2_length" value="0.7"/>
+<xacro:property name="link2_length" value="0.5"/>
 <!--  joint 2   -->
         <joint name="${prefix}joint2" type="${joint2_type}">
           <parent link="${prefix}link1"/>
           <child link="${prefix}link2" />
-          <origin xyz="0 0 ${link1_length}" rpy="0 0 0 "/>
+          <origin xyz="0 ${link1_radius} ${link1_length}" rpy="${-1/2*pi} 0 0 "/>
           <axis xyz="${joint2_axe}"/>
           <xacro:joint_limit joint_type="${joint2_type}" link_length="${link2_length}"/>
@@ -170,5 +170,5 @@
           <parent link="${prefix}link2"/>
           <child link="${prefix}link3" />
-          <origin xyz="0 ${link2_radius} ${link2_length}" rpy="${-1/2*pi} 0 0 "/>
+          <origin xyz="0 -${link2_radius} ${link2_length}" rpy="${1/2*pi} 0 0 "/>
           <axis xyz="${joint3_axe}"/>
           <xacro:joint_limit joint_type="${joint3_type}" link_length="${link3_length}"/>
@@ -194,5 +194,5 @@
         </link>
 <xacro:property name="joint4_type" value="revolute"/>
-<xacro:property name="joint4_axe" value="0 0 1"/>
+<xacro:property name="joint4_axe" value="0 1 0"/>
 <xacro:property name="link4_length" value="0.5"/>
 <!--  joint 4   -->
@@ -200,5 +200,5 @@
           <parent link="${prefix}link3"/>
           <child link="${prefix}link4" />
-          <origin xyz="0 -${link3_radius} ${link3_length}" rpy="${1/2*pi} 0 0 "/>
+          <origin xyz="0 ${link3_radius+link4_radius} ${link3_length}" rpy="0 0 0 "/>
           <axis xyz="${joint4_axe}"/>
           <xacro:joint_limit joint_type="${joint4_type}" link_length="${link4_length}"/>
@@ -224,5 +224,5 @@
         </link>
 <xacro:property name="joint5_type" value="revolute"/>
-<xacro:property name="joint5_axe" value="0 0 1"/>
+<xacro:property name="joint5_axe" value="0 1 0"/>
 <xacro:property name="link5_length" value="0.3"/>
 <!--  joint 5   -->
@@ -230,5 +230,5 @@
           <parent link="${prefix}link4"/>
           <child link="${prefix}link5" />
-          <origin xyz="0 ${link4_radius} ${link4_length}" rpy="${-1/2*pi} 0 0 "/>
+          <origin xyz="0 ${link4_radius+link5_radius} ${link4_length}" rpy="0 0 0 "/>
           <axis xyz="${joint5_axe}"/>
           <xacro:joint_limit joint_type="${joint5_type}" link_length="${link5_length}"/>
@@ -253,17 +253,17 @@
           </xacro:cylinder_inertial>
         </link>
-<xacro:property name="joint6_type" value="prismatic"/>
-<xacro:property name="joint6_axe" value="0 0 1"/>
+<!--<xacro:property name="joint6_type" value="revolute"/>
+<xacro:property name="joint6_axe" value="0 1 0"/>
 <xacro:property name="link6_length" value="0.1"/>
-<!--  joint 6   -->
+  joint 6
         <joint name="${prefix}joint6" type="${joint6_type}">
           <parent link="${prefix}link5"/>
           <child link="${prefix}link6" />
-          <origin xyz="0 0 ${link5_length + link6_radius}" rpy="${-1/2*pi} 0 0 "/>
+          <origin xyz="0 ${link5_radius+link6_radius} ${link5_length}" rpy="0 0 0 "/>
           <axis xyz="${joint6_axe}"/>
           <xacro:joint_limit joint_type="${joint6_type}" link_length="${link6_length}"/>
           <dynamics damping="0.0" friction="0.0"/>
-        </joint>
-    <!-- link 6   -->
+        </joint>  -->
+    <!-- link 6
         <link name="${prefix}link6">
           <visual>
@@ -282,10 +282,10 @@
             <origin xyz="0.0 0.0 ${link6_length / 2 }" rpy="0 0 0" />
           </xacro:cylinder_inertial>
-        </link>
+        </link>-->
         <!-- Sprayer joint - fictive joint -->
         <joint name="fake_joint" type="revolute">
-            <parent link="${prefix}link6" />
+            <parent link="${prefix}link5" />
             <child link = "camera_link" />
-            <origin xyz="0.0  0.0 ${link6_length}" rpy="0.0 0.0 0" />
+            <origin xyz="0.0  0.0 ${link5_length}" rpy="0.0 0.0 0" />
             <axis xyz="0 0 1"/>
             <xacro:joint_limit joint_type="revolute" link_length="0.1"/>

File: man_gazebo/urdf/6dof/arms/_roll_z_0_1_pris_z_0_5_roll_y_0_5_roll_y_0_5_roll_y_0_3_pris_y_0_1.urdf.xacro (robot description, xacro)
@@ -4,4 +4,10 @@
         <xacro:include filename="$(find man_gazebo)/urdf/6dof/transmission_6dof.xacro" />
         <xacro:include filename="$(find man_gazebo)/urdf/gazebo.xacro" />
+        <link name="world" />
+        <joint name="world_joint" type="fixed">
+            <parent link="world" />
+            <child link = "base_link" />
+            <origin xyz="0 0 0" rpy="0.0 0.0 0.0" />
+        </joint>
         <xacro:macro name="cylinder_inertial" params="radius length mass *origin">
         <inertial>
@@ -33,6 +39,6 @@
         <xacro:property name="link0_mass" value="7" />
         <xacro:property name="link1_mass" value="3.7" />
-        <xacro:property name="link2_mass" value="5.12043" />
-        <xacro:property name="link3_mass" value="2.19447" />
+        <xacro:property name="link2_mass" value="3.65745" />
+        <xacro:property name="link3_mass" value="3.65745" />
         <xacro:property name="link4_mass" value="3.65745" />
         <xacro:property name="link5_mass" value="2.19447" />
@@ -45,10 +51,4 @@
         <xacro:property name="link5_radius" value="0.030" />
         <xacro:property name="link6_radius" value="0.025" />
-        <link name="world" />
-          <joint name="world_joint" type="fixed">
-            <parent link="world" />
-            <child link = "base_link" />
-            <origin xyz="0 0 0" rpy="0.0 0.0 0.0" />
-          </joint>
         <!-- Base Link -->
         <link name="${prefix}base_link" >
@@ -135,5 +135,5 @@
 <xacro:property name="joint2_type" value="prismatic"/>
 <xacro:property name="joint2_axe" value="0 0 1"/>
-<xacro:property name="link2_length" value="0.7"/>
+<xacro:property name="link2_length" value="0.5"/>
 <!--  joint 2   -->
         <joint name="${prefix}joint2" type="${joint2_type}">
@@ -165,5 +165,5 @@
 <xacro:property name="joint3_type" value="revolute"/>
 <xacro:property name="joint3_axe" value="0 0 1"/>
-<xacro:property name="link3_length" value="0.3"/>
+<xacro:property name="link3_length" value="0.5"/>
 <!--  joint 3   -->
         <joint name="${prefix}joint3" type="${joint3_type}">
@@ -309,14 +309,5 @@
           </xacro:cylinder_inertial>
         </link>
-        <!-- ee link -->
-        <link name="${prefix}ee_link">
-          <collision>
-            <geometry>
-              <box size="0.01 0.01 0.01"/>
-            </geometry>
-            <origin rpy="0 0 0" xyz="0 0 0.005"/>
-          </collision>
-        </link>
-            <!-- ee joint -->
+        <!-- ee joint -->
         <joint name="${prefix}ee_fixed_joint" type="fixed">
           <parent link="camera_link" />
@@ -324,4 +315,13 @@
           <origin xyz="0.0  0.0 0.01" rpy="0.0 0.0 0" />
         </joint>
+        <!-- ee link -->
+        <link name="${prefix}ee_link">
+          <collision>
+            <geometry>
+              <box size="0.01 0.01 0.01"/>
+            </geometry>
+            <origin rpy="0 0 0" xyz="0 0 0.005"/>
+          </collision>
+        </link>
             <xacro:arm_transmission prefix="${prefix}" />
             <xacro:arm_gazebo prefix="${prefix}" />
